File: Esp32-card-first-Test/AlimentationSheet.kicad_sch (KiCad schematic)
At the start: 5 parts, among them J6 Conn_01x02_Pin, J7 Conn_01x02_Socket, U5 L7805

Commit message: .
Parts:
- removed C1, C2: C, Capacitor_THT:CP_Radial_D4.0mm_P1.50mm, symbol Device:C
- removed J7: Conn_01x02_Socket, TerminalBlock:TerminalBlock_bornier-2_P5.08mm, symbol Connector:Conn_01x02_Socket
- removed U5: L7805, Package_TO_SOT_THT:TO-220-3_Vertical, symbol Regulator_Linear:L7805
