File: Hardware/Esp32-card-first-Test/GPIO_Extender.kicad_sch (KiCad schematic)
At the start: 6 parts, among them J12 Conn_01x05_Pin, J14 Conn_01x06_Pin, J9 Conn_01x05_Pin, U1 74HC595, U2 74HC595, U4 74HC4051

Commit message: pcb
Parts:
- removed J9: Conn_01x05_Pin, Connector_PinHeader_2.54mm:PinHeader_1x05_P2.54mm_Vertical, symbol Connector:Conn_01x05_Pin
- added J1: Conn_01x15_Pin, Connector_PinHeader_2.54mm:PinHeader_1x15_P2.54mm_Vertical, symbol Connector:Conn_01x15_Pin
- added J9: Conn_01x10_Pin, Connector_PinHeader_2.54mm:PinHeader_1x10_P2.54mm_Vertical, symbol Connector:Conn_01x10_Pin
- added U3: 74HC4051, Package_DIP:DIP-16_W7.62mm, symbol 74xx:74HC4051
- J14: footprint Connector_PinHeader_2.54mm:PinHeader_1x06_P2.54mm_Horizontal -> Connector_PinHeader_2.54mm:PinHeader_1x06_P2.54mm_Vertical
Connections:
- net M2_Pin_Dir1 is gone; now on an unnamed net: U1.2 (QC)
- net 3v3: now also U3.16 (VCC)
- net Analog_Pin1: no longer U4.3 (A)
- net Clock: no longer J12.4 (Pin_4), U1.11 (SRCLK), U2.11 (SRCLK)
- net Data: no longer U1.14 (SER)
- net GND: no longer J12.2 (Pin_2), J14.2 (Pin_2), U1.13 (~{OE}), U1.8 (GND), U2.13 (~{OE}), U2.8 (GND), U4.6 (~{E}), U4.7 (VEE), U4.8 (GND)
- net Trig: no longer J12.3 (Pin_3), U1.12 (RCLK), U2.12 (RCLK)
- net at J14.3 (Pin_3): now also J12.3 (Pin_3), U1.12 (RCLK), U2.12 (RCLK); no longer U2.2 (QC)
- net at J14.4 (Pin_4): now also J12.4 (Pin_4), U1.11 (SRCLK), U2.11 (SRCLK); no longer U2.1 (QB)
- net at J14.5 (Pin_5): now also U1.14 (SER); no longer U2.15 (QA)
- net at J14.6 (Pin_6): now also U4.3 (A); no longer U4.13 (A0)
- net at U2.3 (QD): now also J9.5 (Pin_5)
- net at U2.4 (QE): now also J9.4 (Pin_4)
- net at U2.5 (QF): now also J9.3 (Pin_3)
- net at U2.6 (QG): now also J9.2 (Pin_2)
- net at U2.7 (QH): now also J9.1 (Pin_1)
- net at U1.5 (QF): now also U3.9 (S2); no longer U4.10 (S1)
- net at U1.4 (QE): now also U3.10 (S1); no longer U4.11 (S0)
- net at U4.9 (S2): no longer U1.6 (QG)
- net at U1.7 (QH): now also J9.9 (Pin_9)
- net Capteur_Autre_1: no longer names the net of U4.2 (A6)
- net Capteur_Autre_1: now also J1.10 (Pin_10)
- net Capteur_Autre_2: no longer names the net of U4.4 (A7)
- net Capteur_Autre_2: now also J1.9 (Pin_9)
- net Capteur_Force_1: no longer names the net of U4.14 (A1)
- net Capteur_Force_1: now also J1.15 (Pin_15)
- net Capteur_Force_2: no longer names the net of U4.15 (A2)
- net Capteur_Force_2: now also J1.14 (Pin_14)
- net Capteur_Force_3: no longer names the net of U4.12 (A3)
- net Capteur_Force_3: now also J1.13 (Pin_13)
- net Capteur_Hall_1: no longer names the net of U4.1 (A4)
- net Capteur_Hall_1: now also J1.12 (Pin_12)
- net Capteur_Hall_2: no longer names the net of U4.5 (A5)
- net Capteur_Hall_2: now also J1.11 (Pin_11)
- net M1_Pin_Dir1: no longer names the net of U1.15 (QA)
- net M1_Pin_Dir1: now also U4.11 (S0)
- net M1_Pin_Dir2: no longer names the net of U1.1 (QB)
- net M1_Pin_Dir2: now also U4.10 (S1)
- net M2_Pin_Dir2: no longer names the net of U1.3 (QD)
- net M2_Pin_Dir2: now also U3.11 (S0)
- new net: J1.1 (Pin_1), U3.4 (A7)
- new net: J1.2 (Pin_2), U3.2 (A6)
- new net: J1.3 (Pin_3), U3.5 (A5)
- new net: J1.4 (Pin_4), U3.1 (A4)
- new net: J1.5 (Pin_5), U3.12 (A3)
- new net: J1.6 (Pin_6), U3.15 (A2)
- new net: J1.7 (Pin_7), U3.14 (A1)
- new net: J1.8 (Pin_8), U3.13 (A0)
- new net: J12.2 (Pin_2), J14.2 (Pin_2), U1.13 (~{OE}), U1.8 (GND), U2.13 (~{OE}), U2.8 (GND), U3.6 (~{E}), U3.7 (VEE), U3.8 (GND), U4.6 (~{E}), U4.7 (VEE), U4.8 (GND)
- new net: U3.3 (A), U4.13 (A0)
- new net: J9.7 (Pin_7), U2.1 (QB)
- new net: J9.8 (Pin_8), U2.15 (QA)
- new net: J9.6 (Pin_6), U2.2 (QC)
- new net: J9.10 (Pin_10), U1.6 (QG)

Commit message: update
Parts:
- removed J1: Conn_01x15_Pin, Connector_PinHeader_2.54mm:PinHeader_1x15_P2.54mm_Vertical, symbol Connector:Conn_01x15_Pin
- added J1: Conn_01x07_Pin, Connector_PinHeader_2.54mm:PinHeader_1x07_P2.54mm_Vertical, symbol Connector:Conn_01x07_Pin
- added J15: Conn_01x08_Pin, Connector_PinHeader_2.54mm:PinHeader_1x08_P2.54mm_Vertical, symbol Connector:Conn_01x08_Pin
Connections:
- net at U3.4 (A7): now also J15.1 (Pin_1)
- net at U4.2 (A6): now also J1.2 (Pin_2)
- net at U4.5 (A5): now also J1.3 (Pin_3)
- net at U4.1 (A4): now also J1.4 (Pin_4)
- net at U4.12 (A3): now also J1.5 (Pin_5)
- net at U4.15 (A2): now also J1.6 (Pin_6)
- net at U4.14 (A1): now also J1.7 (Pin_7)
- net at U3.2 (A6): now also J15.2 (Pin_2)
- net at U3.5 (A5): now also J15.3 (Pin_3)
- net at U3.1 (A4): now also J15.4 (Pin_4)
- net at U3.12 (A3): now also J15.5 (Pin_5)
- net at U3.15 (A2): now also J15.6 (Pin_6)
- net at U3.14 (A1): now also J15.7 (Pin_7)
- net at U3.13 (A0): now also J15.8 (Pin_8)
- net at U4.4 (A7): now also J1.1 (Pin_1)
Changed lines of the file:
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@@
-	)
-	(symbol
-		(lib_id "Connector:Conn_01x15_Pin")
-		(at 231.14 82.55 180)
-		(unit 1)
-		(exclude_from_sim no)
-		(in_bom yes)
-		(on_board yes)
-		(dnp no)
-		(fields_autoplaced yes)
-		(property "Reference" "J1"
-			(at 232.41 81.2799 0)
-			(effects
-				(font
-					(size 1.27 1.27)
-				)
-				(justify right)
-			)
-		)
-		(property "Value" "Conn_01x15_Pin"
-			(at 232.41 83.8199 0)
-			(effects
-				(font
-					(size 1.27 1.27)
-				)
-				(justify right)
-			)
-		)
-		(property "Footprint" "Connector_PinHeader_2.54mm:PinHeader_1x15_P2.54mm_Vertical"
-			(at 231.14 82.55 0)
-			(effects
-				(font
-					(size 1.27 1.27)
-				)
-				(hide yes)
-			)
-		)
-		(property "Datasheet" "~"
-			(at 231.14 82.55 0)
-			(effects
-				(font
-					(size 1.27 1.27)
-				)
-				(hide yes)
-			)
-		)
-		(property "Description" "Generic connector, single row, 01x15, script generated"
-			(at 231.14 82.55 0)
-			(effects
-				(font
-					(size 1.27 1.27)
-				)
-				(hide yes)
-			)
-		)
-		(pin "10"
-		)
-		(pin "9"
-		)
-		(pin "11"
-		)
-		(pin "5"
-		)
-		(pin "14"
-		)
-		(pin "12"
-		)
-		(pin "15"
-		)
-		(pin "7"
-		)
-		(pin "3"
-		)
-		(pin "4"
-		)
-		(pin "13"
-		)
-		(pin "6"
-		)
-		(pin "2"
-		)
-		(pin "1"
-		)
-		(pin "8"
-		)
-		(instances
-			(project ""
-				(path "/00172638-8708-4530-9462-7b89510d184e/e79c3383-5a03-4763-a384-7173bf81024c"
-					(reference "J1")
-					(unit 1)
-				)
-			)
-		)
 	)
 	(symbol
@@
 	)
 	(symbol
+		(lib_id "Connector:Conn_01x08_Pin")
+		(at 231.14 92.71 180)
+		(unit 1)
+		(exclude_from_sim no)
+		(in_bom yes)
+		(on_board yes)
+		(dnp no)
+		(fields_autoplaced yes)
+		(property "Reference" "J15"
+			(at 232.41 90.1699 0)
+			(effects
+				(font
+					(size 1.27 1.27)
+				)
+				(justify right)
+			)
+		)
+		(property "Value" "Conn_01x08_Pin"
+			(at 232.41 92.7099 0)
+			(effects
+				(font
+					(size 1.27 1.27)
+				)
+				(justify right)
+			)
+		)
+		(property "Footprint" "Connector_PinHeader_2.54mm:PinHeader_1x08_P2.54mm_Vertical"
+			(at 231.14 92.71 0)
+			(effects
+				(font
+					(size 1.27 1.27)
+				)
+				(hide yes)
+			)
+		)
+		(property "Datasheet" "~"
+			(at 231.14 92.71 0)
+			(effects
+				(font
+					(size 1.27 1.27)
+				)
+				(hide yes)
+			)
+		)
+		(property "Description" "Generic connector, single row, 01x08, script generated"
+			(at 231.14 92.71 0)
+			(effects
+				(font
+					(size 1.27 1.27)
+				)
+				(hide yes)
+			)
+		)
+		(pin "1"
+		)
+		(pin "6"
+		)
+		(pin "4"
+		)
+		(pin "3"
+		)
+		(pin "5"
+		)
+		(pin "8"
+		)
+		(pin "7"
+		)
+		(pin "2"
+		)
+		(instances
+			(project ""
+				(path "/00172638-8708-4530-9462-7b89510d184e/e79c3383-5a03-4763-a384-7173bf81024c"
+					(reference "J15")
+					(unit 1)
+				)
+			)
+		)
+	)
+	(symbol
 		(lib_id "Connector:Conn_01x05_Pin")
 		(at 140.97 156.21 180)
@@
 					(unit 1)
 				)
+			)
+		)
+	)
+	(symbol
+		(lib_id "Connector:Conn_01x07_Pin")
+		(at 231.14 72.39 180)
+		(unit 1)
+		(exclude_from_sim no)
+		(in_bom yes)
+		(on_board yes)
+		(dnp no)
+		(fields_autoplaced yes)
+		(property "Reference" "J1"
+			(at 232.41 71.1199 0)
+			(effects
+				(font
+					(size 1.27 1.27)
+				)
+				(justify right)
+			)
+		)
+		(property "Value" "Conn_01x07_Pin"
+			(at 232.41 73.6599 0)
+			(effects
+				(font
+					(size 1.27 1.27)
+				)
+				(justify right)
+			)
+		)
+		(property "Footprint" "Connector_PinHeader_2.54mm:PinHeader_1x07_P2.54mm_Vertical"
+			(at 231.14 72.39 0)
+			(effects
+				(font
+					(size 1.27 1.27)
+				)
+				(hide yes)
+			)
+		)
+		(property "Datasheet" "~"
+			(at 231.14 72.39 0)
+			(effects
+				(font
+					(size 1.27 1.27)
+				)
+				(hide yes)
+			)
+		)
+		(property "Description" "Generic connector, single row, 01x07, script generated"
+			(at 231.14 72.39 0)
+			(effects
+				(font
+					(size 1.27 1.27)
+				)
+				(hide yes)
+			)
+		)
+		(pin "3"
+		)
+		(pin "1"
+		)
+		(pin "5"
+		)
+		(pin "2"
+		)
+		(pin "7"
+		)
+		(pin "4"
+		)
+		(pin "6"
+		)
+		(instances
+			(project ""
+				(path "/00172638-8708-4530-9462-7b89510d184e/e79c3383-5a03-4763-a384-7173bf81024c"
+					(reference "J1")
+					(unit 1)
+				)
